File: RingShield.brd (EAGLE design)
At the start: 136 x 30 mm, 37 parts, among them U1 LED-ADDRESSABLE16MM, U10 LED-ADDRESSABLE16MM, U11 LED-ADDRESSABLE16MM, U12 LED-ADDRESSABLE16MM, U13 LED-ADDRESSABLE16MM, U14 LED-ADDRESSABLE16MM, U15 LED-ADDRESSABLE16MM, U16 LED-ADDRESSABLE16MM, U17 LED-ADDRESSABLE16MM, U18 LED-ADDRESSABLE16MM, U19 LED-ADDRESSABLE16MM, U2 LED-ADDRESSABLE16MM, U20 LED-ADDRESSABLE16MM, U21 LED-ADDRESSABLE16MM, U22 LED-ADDRESSABLE16MM, U23 LED-ADDRESSABLE16MM, U24 LED-ADDRESSABLE16MM, U25 LED-ADDRESSABLE16MM, U26 LED-ADDRESSABLE16MM, U27 LED-ADDRESSABLE16MM, U28 LED-ADDRESSABLE16MM, U29 LED-ADDRESSABLE16MM, U3 LED-ADDRESSABLE16MM, U30 LED-ADDRESSABLE16MM, U4 LED-ADDRESSABLE16MM, U5 LED-ADDRESSABLE16MM, U6 LED-ADDRESSABLE16MM, U7 LED-ADDRESSABLE16MM, U8 LED-ADDRESSABLE16MM, U9 LED-ADDRESSABLE16MM

Commit message: Adding v1.4
Parts:
- removed U1, U10, U11, U12, U13, U14, U15, U16, U17, U18, U19, U2, U20, U21, U22, U23, U24, U25, U26, U27, U28, U29, U3, U30, U4, U5, U6, U7, U8, U9: LED-ADDRESSABLE16MM, ALBERT:LED-WS2812B-2020-RING
- added D1, D10, D11, D12, D13, D14, D15, D16, D17, D18, D19, D2, D20, D3, D4, D5, D6, D7, D8, D9: WS2812B2020, WS2812B2020:LED_WS2812B2020
- added PCB_CONNECTOR: (no value), pinhead:1X03/90
- moved H3 152.6 mm to (41.0, 71.8)
- moved H4 152.4 mm to (41.5, 63.1)
- moved 5V_RELAY 108.3 mm to (29.2, 100.1), flipped to the bottom, turned to 90 degrees
- moved LEFT_SIDE 93.7 mm to (28.0, 65.0), flipped to the bottom, turned to 90 degrees
- moved R1 85.3 mm to (22.8, 28.8), turned to 315 degrees
- moved JP3 83.4 mm to (56.4, 36.1), flipped to the bottom, turned to 90 degrees
- moved RIGHT_SIDE 59.3 mm to (10.0, 65.0), flipped to the bottom, turned to 270 degrees
Connections:
- removed net 5V_OUT: 5V_RELAY.A1, U1.+, U10.+, U2.+, U3.+, U4.+, U5.+, U6.+, U7.+, U8.+, U9.+
- removed net N$18: U12.DO, U13.DI
- removed net N$23: U20.DO, U21.DI
- removed net N$24: U21.DO, U22.DI
- removed net N$25: U22.DO, U23.DI
- removed net N$26: U23.DO, U24.DI
- removed net N$27: U24.DO, U25.DI
- removed net N$28: U25.DO, U26.DI
- removed net N$29: U26.DO, U27.DI
- removed net N$30: U27.DO, U28.DI
- removed net N$31: U28.DO, U29.DI
- removed net N$32: U29.DO, U30.DI
- new net DO: D20.1, PCB_CONNECTOR.2
- new net N$9: D10.3, D9.1
- net +5V: now also 5V_RELAY.A1, D1.4, D10.4, D11.4, D12.4, D13.4, D14.4, D15.4, D16.4, D17.4, D18.4, D19.4, D2.4, D20.4, D3.4, D4.4, D5.4, D6.4, D7.4, D8.4, D9.4, PCB_CONNECTOR.3; no longer U11.+, U12.+, U13.+, U14.+, U15.+, U16.+, U17.+, U18.+, U19.+, U20.+, U21.+, U22.+, U23.+, U24.+, U25.+, U26.+, U27.+, U28.+, U29.+, U30.+
- net GND: now also D1.2, D10.2, D11.2, D12.2, D13.2, D14.2, D15.2, D16.2, D17.2, D18.2, D19.2, D2.2, D20.2, D3.2, D4.2, D5.2, D6.2, D7.2, D8.2, D9.2, PCB_CONNECTOR.1; no longer U1.GND, U10.GND, U11.GND, U12.GND, U13.GND, U14.GND, U15.GND, U16.GND, U17.GND, U18.GND, U19.GND, U2.GND, U20.GND, U21.GND, U22.GND, U23.GND, U24.GND, U25.GND, U26.GND, U27.GND, U28.GND, U29.GND, U3.GND, U30.GND, U4.GND, U5.GND, U6.GND, U7.GND, U8.GND, U9.GND
- net N$1: now also D1.3, R1.2; no longer U1.DO, U2.DI
- net N$10: now also D8.1, D9.3; no longer U7.DO, U8.DI
- net N$11: now also D7.1, D8.3; no longer U8.DO, U9.DI
- net N$12: now also D6.1, D7.3; no longer U10.DI, U9.DO
- net N$13: now also D14.1, D15.3; no longer U10.DO, U11.DI
- net N$14: now also D13.1, D14.3; no longer U15.DO, U16.DI
- net N$15: now also D12.1, D13.3; no longer U16.DO, U17.DI
- net N$16: now also D11.1, D12.3; no longer U17.DO, U18.DI
- net N$17: now also D10.1, D11.3; no longer U11.DO, U12.DI
- net N$19: now also D17.1, D18.3; no longer U13.DO, U14.DI
- net N$2: now also D1.1, D2.3; no longer U2.DO, U3.DI
- net N$20: now also D16.1, D17.3; no longer U14.DO, U15.DI
- net N$21: now also D15.1, D16.3; no longer U18.DO, U19.DI
- net N$22: now also D19.1, D20.3; no longer U19.DO, U20.DI
- net N$3: now also D2.1, D3.3; no longer U3.DO, U4.DI
- net N$4: now also D3.1, D4.3; no longer U4.DO, U5.DI
- net N$5: now also D4.1, D5.3; no longer U5.DO, U6.DI
- net N$6: now also D5.1, D6.3; no longer U6.DO, U7.DI
- net N$7: now also D18.1, D19.3; no longer R1.2, U1.DI
Routing:
- net +5V: track 0.00 -> 215.0 mm
- net GND: track 0.00 -> 173.7 mm
- net DO: track 0.00 -> 16.2 mm
- net N$4: track 0.00 -> 11.3 mm
- net N$5: track 0.00 -> 9.14 mm
- net N$3: track 0.00 -> 8.61 mm
- net N$6: track 0.00 -> 8.52 mm
- net N$2: track 0.00 -> 7.55 mm
Other:
- board size 136 x 30 mm -> 70 x 140 mm
